File: pcb/module-b/module-b.kicad_pcb (KiCad board)
At the start: 2 copper layers, 76 x 176 mm, 14 parts, among them J1 Conn_01x06, J2 Conn_01x06, SW1 RotaryEncoder_Switch_MP, SW2 RotaryEncoder_Switch_MP, SW3 RotaryEncoder_Switch_MP, U1 ESP32-C3, U2 MCP23S17_SO

Commit message: 3V net should not be shared across the bus
Connections:
- C1 pad 1: 3V3 -> Net-(U1-V3V)
- J1 pad 3: 3V3 -> Net-(J1-Pin_3)
- J2 pad 3: 3V3 -> Net-(J1-Pin_3)
- U1 pad 3: 3V3 -> Net-(U1-V3V)
- U2 pad 9: 3V3 -> Net-(U1-V3V)
Routing:
- net 3V3: track 94.0 -> 0.00 mm, vias 1 -> 0
- net Net-(J1-Pin_3): track 0.00 -> 69.1 mm
- net Net-(U1-V3V): track 0.00 -> 12.7 mm
Changed lines of the file:
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@@
 	(net 29 "GND")
 	(net 30 "5V")
-	(net 31 "3V3")
+	(net 31 "Net-(U1-V3V)")
 	(net 32 "/SLC")
 	(net 33 "/SDA")
@@
 	(net 36 "unconnected-(U2-GPA3-Pad24)")
 	(net 37 "unconnected-(U2-GPB6-Pad7)")
+	(net 38 "Net-(J1-Pin_3)")
 	(footprint "MountingHole:MountingHole_2.2mm_M2"
 		(layer "F.Cu")
@@
 			(layers "*.Cu" "*.Mask")
 			(remove_unused_layers no)
-			(net 31 "3V3")
+			(net 38 "Net-(J1-Pin_3)")
 			(pinfunction "Pin_3")
 			(pintype "passive")
@@
 			(layers "*.Cu" "*.Mask")
 			(remove_unused_layers no)
-			(net 31 "3V3")
+			(net 38 "Net-(J1-Pin_3)")
 			(pinfunction "Pin_3")
 			(pintype "passive")
@@
 			(layers "B.Cu" "B.Mask" "B.Paste")
 			(roundrect_rratio 0.188679)
-			(net 31 "3V3")
+			(net 31 "Net-(U1-V3V)")
 			(pintype "passive")
 		)
@@
 			(layers "B.Cu" "B.Mask" "B.Paste")
 			(roundrect_rratio 0.25)
-			(net 31 "3V3")
+			(net 31 "Net-(U1-V3V)")
 			(pinfunction "VDD")
 			(pintype "power_in")
@@
 			(size 3 1.5)
 			(layers "B.Cu" "B.Mask" "B.Paste")
-			(net 31 "3V3")
+			(net 31 "Net-(U1-V3V)")
 			(pinfunction "V3V")
 			(pintype "power_out")
@@
 	)
 	(segment
-		(start 145.0125 46.274)
-		(end 174.3225 46.274)
-		(width 0.5)
-		(layer "F.Cu")
-		(net 31)
-	)
-	(segment
-		(start 105.1875 46.274)
-		(end 145.0125 46.274)
-		(width 0.5)
-		(layer "F.Cu")
-		(net 31)
-	)
-	(segment
-		(start 174.3225 46.274)
-		(end 174.3325 46.264)
-		(width 0.5)
-		(layer "F.Cu")
-		(net 31)
-	)
-	(via
-		(at 145.0125 46.274)
-		(size 0.6)
-		(drill 0.3)
-		(layers "F.Cu" "B.Cu")
-		(net 31)
-	)
-	(segment
 		(start 144.9625 34.1065)
 		(end 148.08 34.1065)
@@
 	)
 	(segment
-		(start 144.9625 46.224)
-		(end 144.9625 34.1065)
-		(width 0.5)
-		(layer "B.Cu")
-		(net 31)
-	)
-	(segment
 		(start 138.64 27.784)
 		(end 138.0525 27.784)
@@
 	)
 	(segment
-		(start 145.0125 46.274)
-		(end 144.9625 46.224)
-		(width 0.5)
-		(layer "B.Cu")
-		(net 31)
-	)
-	(segment
 		(start 148.08 34.1065)
 		(end 148.1125 34.139)
@@
 		(net 33)
 	)
+	(segment
+		(start 105.1975 46.264)
+		(end 105.1875 46.274)
+		(width 0.2)
+		(layer "F.Cu")
+		(net 38)
+	)
+	(segment
+		(start 174.3325 46.264)
+		(end 105.1975 46.264)
+		(width 0.2)
+		(layer "F.Cu")
+		(net 38)
+	)
 	(zone
