File: pcb/module-b/module-b.kicad_sch (KiCad schematic)
At the start: 14 parts, among them J1 Conn_01x06, J2 Conn_01x06, SW1 RotaryEncoder_Switch_MP, SW2 RotaryEncoder_Switch_MP, SW3 RotaryEncoder_Switch_MP, U1 ESP32-C3, U2 MCP23S17_SO

Commit message: 3V net should not be shared across the bus
Connections:
- net 3V3: no longer names the net of C1.1, U1.3 (V3V), U2.9 (VDD)
- net 3V3: no longer J1.3 (Pin_3), J2.3 (Pin_3)
- new net: J1.3 (Pin_3), J2.3 (Pin_3)
Changed lines of the file:
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@@
-	)
-	(junction
-		(at 74.93 50.8)
-		(diameter 0)
-		(color 0 0 0 0)
 	)
 	(junction
@@
 	)
 	(junction
-		(at 74.93 36.83)
-		(diameter 0)
-		(color 0 0 0 0)
-	)
-	(junction
 		(at 161.29 113.03)
 		(diameter 0)
@@
 	)
 	(junction
-		(at 82.55 36.83)
-		(diameter 0)
-		(color 0 0 0 0)
-	)
-	(junction
 		(at 180.34 101.6)
 		(diameter 0)
@@
 	(wire
 		(pts
-			(xy 55.88 36.83) (xy 74.93 36.83)
-		)
-		(stroke
-			(width 0)
-			(type default)
-		)
-	)
-	(wire
-		(pts
 			(xy 340.36 93.98) (xy 240.03 93.98)
 		)
@@
 	(wire
 		(pts
-			(xy 82.55 36.83) (xy 102.87 36.83)
+			(xy 55.88 36.83) (xy 102.87 36.83)
 		)
 		(stroke
@@
 	(wire
 		(pts
-			(xy 74.93 64.77) (xy 111.76 64.77)
+			(xy 109.22 64.77) (xy 111.76 64.77)
 		)
 		(stroke
@@
 	(wire
 		(pts
-			(xy 74.93 64.77) (xy 74.93 50.8)
+			(xy 109.22 64.77) (xy 109.22 50.8)
 		)
 		(stroke
@@
 	(wire
 		(pts
-			(xy 74.93 50.8) (xy 161.29 50.8)
+			(xy 109.22 50.8) (xy 161.29 50.8)
 		)
 		(stroke
@@
 	(wire
 		(pts
-			(xy 82.55 24.13) (xy 82.55 36.83)
-		)
-		(stroke
-			(width 0)
-			(type default)
-		)
-	)
-	(wire
-		(pts
 			(xy 198.12 113.03) (xy 180.34 113.03)
 		)
@@
 	(wire
 		(pts
-			(xy 74.93 36.83) (xy 82.55 36.83)
-		)
-		(stroke
-			(width 0)
-			(type default)
-		)
-	)
-	(wire
-		(pts
 			(xy 274.32 60.96) (xy 278.13 60.96)
 		)
@@
 		(pts
 			(xy 100.33 77.47) (xy 100.33 86.36)
-		)
-		(stroke
-			(width 0)
-			(type default)
-		)
-	)
-	(wire
-		(pts
-			(xy 74.93 36.83) (xy 74.93 50.8)
 		)
 		(stroke
@@
 	(label "5V"
 		(at 57.15 31.75 0)
-		(effects
-			(font
-				(size 1.27 1.27)
-			)
-			(justify left bottom)
-		)
-	)
-	(label "3V3"
-		(at 57.15 36.83 0)
 		(effects
 			(font
@@
 				)
 				(justify left)
-				(hide yes)
-			)
-		)
-	)
-	(global_label "3V3"
-		(shape input)
-		(at 82.55 24.13 90)
-		(fields_autoplaced yes)
-		(effects
-			(font
-				(size 1.27 1.27)
-			)
-			(justify left)
-		)
-		(property "Intersheetrefs" "${INTERSHEET_REFS}"
-			(at 82.55 17.6372 90)
-			(effects
-				(font
-					(size 1.27 1.27)
-				)
-				(justify left)
-				(hide yes)
-			)
-		)
-	)
-	(global_label "3V3"
-		(shape input)
-		(at 20.32 34.29 270)
-		(fields_autoplaced yes)
-		(effects
-			(font
-				(size 1.27 1.27)
-			)
-			(justify right)
-		)
-		(property "Intersheetrefs" "${INTERSHEET_REFS}"
-			(at 20.32 40.7828 90)
-			(effects
-				(font
-					(size 1.27 1.27)
-				)
-				(justify right)
 				(hide yes)
 			)
@@
 	)
 	(symbol
+		(lib_id "power:PWR_FLAG")
+		(at 20.32 52.07 90)
+		(unit 1)
+		(exclude_from_sim no)
+		(in_bom yes)
+		(on_board yes)
+		(dnp no)
+		(fields_autoplaced yes)
+		(property "Reference" "#FLG03"
+			(at 18.415 52.07 0)
+			(effects
+				(font
+					(size 1.27 1.27)
+				)
+				(hide yes)
+			)
+		)
+		(property "Value" "PWR_FLAG"
+			(at 16.51 52.0699 90)
+			(effects
+				(font
+					(size 1.27 1.27)
+				)
+				(justify left)
+			)
+		)
+		(property "Footprint" ""
+			(at 20.32 52.07 0)
+			(effects
+				(font
+					(size 1.27 1.27)
+				)
+				(hide yes)
+			)
+		)
+		(property "Datasheet" "~"
+			(at 20.32 52.07 0)
+			(effects
+				(font
+					(size 1.27 1.27)
+				)
+				(hide yes)
+			)
+		)
+		(property "Description" "Special symbol for telling ERC where power comes from"
+			(at 20.32 52.07 0)
+			(effects
+				(font
+					(size 1.27 1.27)
+				)
+				(hide yes)
+			)
+		)
+		(pin "1"
+		)
+		(instances
+			(project "module-b"
+				(path "/0888bf04-c6c1-4923-af80-2189ee3798b4"
+					(reference "#FLG03")
+					(unit 1)
+				)
+			)
+		)
+	)
+	(symbol
 		(lib_id "Mechanical:MountingHole")
 		(at 34.29 116.84 0)
@@
 					(unit 1)
 				)
-			)
-		)
-	)
-	(symbol
-		(lib_id "power:PWR_FLAG")
-		(at 20.32 34.29 0)
-		(unit 1)
-		(exclude_from_sim no)
-		(in_bom yes)
-		(on_board yes)
-		(dnp no)
-		(fields_autoplaced yes)
-		(property "Reference" "#FLG02"
-			(at 20.32 32.385 0)
-			(effects
-				(font
-					(size 1.27 1.27)
-				)
-				(hide yes)
-			)
-		)
-		(property "Value" "PWR_FLAG"
-			(at 20.32 29.21 0)
-			(effects
-				(font
-					(size 1.27 1.27)
-				)
-			)
-		)
-		(property "Footprint" ""
-			(at 20.32 34.29 0)
-			(effects
-				(font
-					(size 1.27 1.27)
-				)
-				(hide yes)
-			)
-		)
-		(property "Datasheet" "~"
-			(at 20.32 34.29 0)
-			(effects
-				(font
-					(size 1.27 1.27)
-				)
-				(hide yes)
-			)
-		)
-		(property "Description" "Special symbol for telling ERC where power comes from"
-			(at 20.32 34.29 0)
-			(effects
-				(font
-					(size 1.27 1.27)
-				)
-				(hide yes)
-			)
-		)
-		(pin "1"
-		)
-		(instances
-			(project "modular-key-pad"
-				(path "/0888bf04-c6c1-4923-af80-2189ee3798b4"
-					(reference "#FLG02")
-					(unit 1)
-				)
