File: pcb/module-a4/module-a4.kicad_pcb (KiCad board)
At the start: 4 copper layers, 76 x 178 mm, 61 parts, among them J1 Conn_01x06, J2 Conn_01x06, J3 USB_C_Receptacle_USB2.0_16P, SW1 SW_Push, SW10 SW_Push, SW11 SW_Push, SW12 SW_Push, SW13 SW_Push_SPDT, SW14 SW_Push, SW15 SW_Push, SW2 SW_Push, SW3 SW_Push, SW4 SW_Push, SW5 SW_Push, SW6 SW_Push, SW7 SW_Push, SW8 SW_Push, SW9 SW_Push, U1 ESP32-S3-WROOM-1, U2 74AHC541, U3 MCP23S17_SO, U4 74HC165, U5 LD1117-3.3H, U6 AP2151W, U7 USBLC6-2SC6

Commit message: Update module a4
Other:
- board text added: "Mod. A-4, rev. 3"
- board text removed: "Mod. A-2, rev. 2"
