File: pcb/module-c/connector-board-r2/connector-board.kicad_pcb (KiCad board)
At the start: 2 copper layers, 76 x 135 mm, 62 parts, among them J1 Conn_01x06, J2 Conn_01x06, J3 Conn_01x06, J4 Conn_01x06, J5 Conn_01x06, J6 Conn_01x06, J7 F3311A7H121024E200, U2 AP2171W, U3 AP2171W, U6 74CBTLV3861BQ,118

Commit message: Update pcb revisions
Connections:
- U6 pad 12: unconnected-(U6-GND-Pad12) -> GND
Routing:
- net GND: track 46.2 -> 47.3 mm, vias 309 -> 311
