File: pcb/module-c/connector-board-r2/connector-board.kicad_sch (KiCad schematic)
At the start: 62 parts, among them J1 Conn_01x06, J2 Conn_01x06, J3 Conn_01x06, J4 Conn_01x06, J5 Conn_01x06, J6 Conn_01x06, J7 F3311A7H121024E200, U2 AP2171W, U3 AP2171W, U6 74CBTLV3861BQ,118

Commit message: Update pcb revisions
Connections:
- net GND: now also U6.12 (GND)
Changed lines of the file:
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@@
 	)
 	(junction
+		(at 406.4 323.85)
+		(diameter 0)
+		(color 0 0 0 0)
+	)
+	(junction
 		(at 123.19 299.72)
 		(diameter 0)
@@
 	(wire
 		(pts
+			(xy 406.4 323.85) (xy 445.77 323.85)
+		)
+		(stroke
+			(width 0)
+			(type default)
+		)
+	)
+	(wire
+		(pts
 			(xy 364.49 228.6) (xy 420.37 228.6)
 		)
@@
 	(wire
 		(pts
-			(xy 381 323.85) (xy 445.77 323.85)
+			(xy 381 323.85) (xy 406.4 323.85)
 		)
 		(stroke
@@
 	(wire
 		(pts
+			(xy 406.4 318.77) (xy 406.4 323.85)
+		)
+		(stroke
+			(width 0)
+			(type default)
+		)
+	)
+	(wire
+		(pts
 			(xy 67.31 124.46) (xy 151.13 124.46)
 		)
@@
 	(symbol
 		(lib_id "power:PWR_FLAG")
-		(at 49.53 29.21 0)
+		(at 40.64 29.21 0)
 		(unit 1)
 		(body_style 1)
@@
 		(fields_autoplaced yes)
 		(property "Reference" "#FLG01"
-			(at 49.53 27.305 0)
+			(at 40.64 27.305 0)
 			(hide yes)
 			(show_name no)
@@
 		)
 		(property "Value" "PWR_FLAG"
-			(at 49.53 24.13 0)
+			(at 40.64 24.13 0)
 			(show_name no)
 			(do_not_autoplace no)
@@
 		)
 		(property "Footprint" ""
-			(at 49.53 29.21 0)
+			(at 40.64 29.21 0)
 			(hide yes)
 			(show_name no)
@@
 		)
 		(property "Datasheet" ""
-			(at 49.53 29.21 0)
+			(at 40.64 29.21 0)
 			(hide yes)
 			(show_name no)
@@
 		)
 		(property "Description" "Special symbol for telling ERC where power comes from"
-			(at 49.53 29.21 0)
+			(at 40.64 29.21 0)
 			(hide yes)
 			(show_name no)
@@
 	(symbol
 		(lib_id "power:GND")
-		(at 49.53 29.21 0)
+		(at 40.64 29.21 0)
 		(unit 1)
 		(body_style 1)
@@
 		(fields_autoplaced yes)
 		(property "Reference" "#PWR01"
-			(at 49.53 35.56 0)
+			(at 40.64 35.56 0)
 			(hide yes)
 			(show_name no)
@@
 		)
 		(property "Value" "GND"
-			(at 49.53 34.29 0)
+			(at 40.64 34.29 0)
 			(show_name no)
 			(do_not_autoplace no)
@@
 		)
 		(property "Footprint" ""
-			(at 49.53 29.21 0)
+			(at 40.64 29.21 0)
 			(hide yes)
 			(show_name no)
@@
 		)
 		(property "Datasheet" ""
-			(at 49.53 29.21 0)
+			(at 40.64 29.21 0)
 			(hide yes)
 			(show_name no)
@@
 		)
 		(property "Description" "Power symbol creates a global label with name \"GND\" , ground"
-			(at 49.53 29.21 0)
+			(at 40.64 29.21 0)
 			(hide yes)
 			(show_name no)
@@
 	(symbol
 		(lib_id "power:+3.3V")
-		(at 55.88 29.21 180)
+		(at 52.07 29.21 180)
 		(unit 1)
 		(body_style 1)
@@
 		(fields_autoplaced yes)
 		(property "Reference" "#PWR02"
-			(at 55.88 25.4 0)
+			(at 52.07 25.4 0)
 			(hide yes)
 			(show_name no)
@@
 		)
 		(property "Value" "+5V"
-			(at 55.88 34.29 0)
+			(at 52.07 34.29 0)
 			(show_name no)
 			(do_not_autoplace no)
@@
 		)
 		(property "Footprint" ""
-			(at 55.88 29.21 0)
+			(at 52.07 29.21 0)
 			(hide yes)
 			(show_name no)
@@
 		)
 		(property "Datasheet" ""
-			(at 55.88 29.21 0)
+			(at 52.07 29.21 0)
 			(hide yes)
 			(show_name no)
@@
 		)
 		(property "Description" "Power symbol creates a global label with name \"+3.3V\""
-			(at 55.88 29.21 0)
+			(at 52.07 29.21 0)
 			(hide yes)
 			(show_name no)
@@
 	(symbol
 		(lib_id "power:PWR_FLAG")
-		(at 55.88 29.21 0)
+		(at 52.07 29.21 0)
 		(unit 1)
 		(body_style 1)
@@
 		(fields_autoplaced yes)
 		(property "Reference" "#FLG02"
-			(at 55.88 27.305 0)
+			(at 52.07 27.305 0)
 			(hide yes)
 			(show_name no)
@@
 		)
 		(property "Value" "PWR_FLAG"
-			(at 55.88 24.13 0)
+			(at 52.07 24.13 0)
 			(show_name no)
 			(do_not_autoplace no)
@@
 		)
 		(property "Footprint" ""
-			(at 55.88 29.21 0)
+			(at 52.07 29.21 0)
 			(hide yes)
 			(show_name no)
@@
 		)
 		(property "Datasheet" ""
-			(at 55.88 29.21 0)
+			(at 52.07 29.21 0)
 			(hide yes)
 			(show_name no)
@@
 		)
 		(property "Description" "Special symbol for telling ERC where power comes from"
-			(at 55.88 29.21 0)
+			(at 52.07 29.21 0)
 			(hide yes)
 			(show_name no)
