File: pcb/module-c/sub-module-programmer-r1/sub-module-programmer.kicad_pcb (KiCad board)
At the start: 2 copper layers, 127 x 50.8 mm, 25 parts, among them J1 Conn_01x06, J2 Conn_01x03, J3 Conn_01x06, J4 Conn_01x06, J5 Conn_01x06, J6 Conn_01x06, J7 Conn_01x06, J8 Serial Bridge, U1 74AHCT1G125, U4 LD1117S33TR_SOT223

Commit message: Update pcb revisions
Parts:
- added C1: 10uF, Capacitor_SMD:C_1206_3216Metric, F.Cu at (159.7, 57.4)
- added C2: 10uF, Capacitor_SMD:C_1206_3216Metric, F.Cu at (157.1, 57.4)
- added C6: 0.1uF, Capacitor_SMD:C_0603_1608Metric, F.Cu at (167.3, 59.9)
- added C7: 0.1uF, Capacitor_SMD:C_0603_1608Metric, F.Cu at (167.3, 49.5)
- added R1: 1k, Resistor_SMD:R_1206_3216Metric, F.Cu at (163.5, 45.8)
- added R10: 100, Resistor_SMD:R_1206_3216Metric, F.Cu at (114.1, 45.8)
- added R11: 2.2, Resistor_SMD:R_0603_1608Metric, F.Cu at (167.3, 56.8)
- added R12: 2.2, Resistor_SMD:R_0603_1608Metric, F.Cu at (167.3, 52.6)
- added R2: 1k, Resistor_SMD:R_1206_3216Metric, F.Cu at (163.5, 48.3)
- added R3: 1k, Resistor_SMD:R_1206_3216Metric, F.Cu at (163.5, 50.9)
- added R4: 4.7, Resistor_SMD:R_1206_3216Metric, F.Cu at (163.5, 53.4)
- added R5: 4.7, Resistor_SMD:R_1206_3216Metric, F.Cu at (163.5, 56.0)
- added R6: 1k, Resistor_SMD:R_1206_3216Metric, F.Cu at (114.1, 48.3)
- added R7: 220, Resistor_SMD:R_1206_3216Metric, F.Cu at (114.1, 56.0)
- added R8: 220, Resistor_SMD:R_1206_3216Metric, F.Cu at (114.1, 53.4)
- added R9: 220, Resistor_SMD:R_1206_3216Metric, F.Cu at (114.1, 50.9)
Connections:
- J1 pad 2: ~{INT} -> Net-(J1-Pin_2)
- J1 pad 3: BRIDGE_RX -> Net-(J1-Pin_3)
- J1 pad 4: BRIDGE_TX -> Net-(J1-Pin_4)
- J1 pad 5: +5V -> Net-(J1-Pin_5)
- J1 pad 6: +3.3V -> Net-(J1-Pin_6)
- J3 pad 2: ~{RESET} -> Net-(J3-Pin_2)
- J3 pad 3: ~{SS} -> Net-(J3-Pin_3)
- J3 pad 4: MOSI -> Net-(J3-Pin_4)
- J3 pad 5: MISO -> Net-(J3-Pin_5)
- J3 pad 6: SCK -> Net-(J3-Pin_6)
Routing:
- net +5V: track 124.3 -> 95.6 mm, vias 6 -> 4
- net BRIDGE_TX: track 97.0 -> 106.7 mm, vias 2 -> 3
- net SCK: track 106.6 -> 97.5 mm
- net +3.3V: track 96.8 -> 87.9 mm, vias 2 -> 3
- net ~{INT}: track 93.1 -> 84.7 mm
- net ~{RESET}: track 151.4 -> 143.1 mm
- net BRIDGE_RX: track 100.6 -> 108.7 mm, vias 3 -> 4
- net ~{SS}: track 83.8 -> 76.4 mm
- net MOSI: track 91.4 -> 84.0 mm
- net MISO: track 99.0 -> 91.9 mm
- net Net-(J1-Pin_5): track 0.00 -> 6.38 mm
- net Net-(J1-Pin_3): track 0.00 -> 6.38 mm, vias 0 -> 1
- net Net-(J1-Pin_2): track 0.00 -> 6.38 mm
- net Net-(J1-Pin_6): track 0.00 -> 6.34 mm
- net Net-(J1-Pin_4): track 0.00 -> 6.34 mm, vias 0 -> 1
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Other:
- board text removed: "Module"
